Commit message: add livox to urdf

File: go2_description/urdf/go2_description.urdf (robot description, URDF)
Before this commit: robot go2_description, 29 links, 28 joints
Links:
- added link livox_frame
- added link livox_lidar; collision cylinder length=0.09 radius=0.05; visual mesh filename=package://go2_description/dae/livox_mid360.dae
Joints:
- added joint livox_frame_joint: type fixed, parent livox_lidar, child livox_frame, origin xyz=0 0 0.047 rpy=0 0 0, axis 0 0 0
- added joint livox_lidar_joint: type fixed, parent base_link, child livox_lidar, origin xyz=0.155 0 0.09 rpy=0 0.20944 0, axis 0 0 0
